File: kicad/uartusb.kicad_pcb (KiCad board)
At the start: 2 copper layers, 47.8 x 23 mm, 27 parts, among them J1 PIN 1x8R, J2 USB_A, J3 dsr, J4 dcd, J5 cts, J6 ri, U1 PL2303HXA, Y1 HC49U 12Mgh

Commit message: start
Parts:
- moved R2 3.23 mm to (187.4, 97.1)
Routing:
- net /vdd5: track 50.1 -> 53.9 mm
- net Net-(R2-Pad2): track 10.9 -> 8.11 mm
- net /dp: track 9.83 -> 12.5 mm
- net /dm: track 3.99 -> 5.35 mm
Other:
- board size 47.8 x 23 mm -> 46.3 x 23 mm
Changed lines of the file:
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@@
     (links 59)
     (no_connects 0)
-    (area 152.124999 82.524999 200.075001 105.675001)
+    (area 152.124999 82.524999 198.575001 105.675001)
     (thickness 1.6)
     (drawings 4)
-    (tracks 165)
+    (tracks 167)
     (zones 0)
     (modules 27)
@@
   (page A4)
   (layers
-    (0 F.Cu signal hide)
-    (31 B.Cu signal)
+    (0 F.Cu signal)
+    (31 B.Cu signal hide)
     (32 B.Adhes user)
     (33 F.Adhes user)
@@
     (pad_to_mask_clearance 0.2)
     (aux_axis_origin 0 0)
-    (visible_elements FFFCB71F)
+    (visible_elements FFFC771F)
     (pcbplotparams
       (layerselection 0x00030_80000001)
@@
   )
   (module Resistors_SMD:R_0603_HandSoldering (layer F.Cu)
-    (at 188.3 94 180)
+    (at 187.4 97.1 180)
     (descr "Resistor SMD 0603, hand soldering")
     (tags "resistor 0603")
@@
     (fp_line (start -6 -4) (end -6 -21.6) (layer B.SilkS) (width 0.1))
     (fp_line (start -6 -4) (end -6 -9) (layer B.SilkS) (width 0.1))
-    (fp_line (start -6 -9) (end 6 -9) (layer B.SilkS) (width 0.1))
+    (fp_line (start -6 -7) (end 6 -7) (layer B.SilkS) (width 0.1))
     (fp_line (start 6 -9) (end 6 -4) (layer B.SilkS) (width 0.1))
     (fp_line (start 6 -4) (end -6 -4) (layer B.SilkS) (width 0.1))
     (pad 6 thru_hole circle (at 2.25 -4 270) (size 1.5 1.5) (drill 0.8) (layers *.Cu *.Mask))
-    (pad 2 thru_hole circle (at -1 -2 270) (size 1.6 1.6) (drill 0.9) (layers *.Cu *.Mask)
+    (pad 3 thru_hole circle (at -1 -2 270) (size 1.65 1.65) (drill 0.9) (layers *.Cu *.Mask)
+      (net 12 /dp))
+    (pad 2 thru_hole circle (at 1 -2 270) (size 1.65 1.65) (drill 0.9) (layers *.Cu *.Mask)
       (net 10 /dm))
-    (pad 3 thru_hole circle (at 1 -2 270) (size 1.6 1.6) (drill 0.9) (layers *.Cu *.Mask)
-      (net 12 /dp))
-    (pad 1 thru_hole circle (at -3 -2 270) (size 1.6 1.6) (drill 0.9) (layers *.Cu *.Mask)
+    (pad 4 thru_hole circle (at -3.5 -2 270) (size 1.65 1.65) (drill 0.9) (layers *.Cu *.Mask)
+      (net 2 GND))
+    (pad 1 thru_hole circle (at 3.5 -2 270) (size 1.65 1.65) (drill 0.9) (layers *.Cu *.Mask)
       (net 3 /vdd5))
-    (pad 4 thru_hole circle (at 3 -2 270) (size 1.6 1.6) (drill 0.9) (layers *.Cu *.Mask)
-      (net 2 GND))
-    (pad 5 thru_hole circle (at -6 -4 270) (size 3 3) (drill 2) (layers *.Cu *.Mask)
-      (net 2 GND))
-    (pad 5 thru_hole circle (at 6 -4 270) (size 3 3) (drill 2) (layers *.Cu *.Mask)
+    (pad 5 thru_hole circle (at -6 -4 270) (size 3.5 3.5) (drill 2) (layers *.Cu *.Mask)
+      (net 2 GND))
+    (pad 5 thru_hole circle (at 6 -4 270) (size 3.5 3.5) (drill 2) (layers *.Cu *.Mask)
       (net 2 GND))
     (pad 6 thru_hole circle (at -2.25 -4 270) (size 1.5 1.5) (drill 0.8) (layers *.Cu *.Mask))
   )
   (gr_line (start 152.2 105.6) (end 152.2 82.6) (angle 90) (layer Edge.Cuts) (width 0.15))
-  (gr_line (start 200 105.6) (end 152.2 105.6) (angle 90) (layer Edge.Cuts) (width 0.15))
-  (gr_line (start 200 82.6) (end 200 105.6) (angle 90) (layer Edge.Cuts) (width 0.15))
-  (gr_line (start 152.2 82.6) (end 200 82.6) (angle 90) (layer Edge.Cuts) (width 0.15))
+  (gr_line (start 198.5 105.6) (end 152.2 105.6) (angle 90) (layer Edge.Cuts) (width 0.15))
+  (gr_line (start 198.5 82.6) (end 198.5 105.6) (angle 90) (layer Edge.Cuts) (width 0.15))
+  (gr_line (start 152.2 82.6) (end 198.5 82.6) (angle 90) (layer Edge.Cuts) (width 0.15))
   (segment (start 159.05 101.45) (end 159.05 100.425) (width 0.3) (layer F.Cu) (net 1))
   (segment (start 159.05 100.425) (end 159.1 100.375) (width 0.3) (layer F.Cu) (net 1))
@@
   (segment (start 176.3 93.448) (end 177.083 92.665) (width 0.3) (layer F.Cu) (net 2))
   (segment (start 175.9 93.848) (end 176.3 93.448) (width 0.3) (layer F.Cu) (net 2))
-  (segment (start 187.2 92.3) (end 189.75 92.3) (width 0.3) (layer B.Cu) (net 3) (status C00000))
-  (segment (start 189.75 92.3) (end 189.8 92.35) (width 0.3) (layer B.Cu) (net 3) (status C00000))
-  (segment (start 193.1 91.3) (end 190.85 91.3) (width 0.3) (layer B.Cu) (net 3) (status 400000))
-  (segment (start 190.85 91.3) (end 189.8 92.35) (width 0.3) (layer B.Cu) (net 3) (status 800000))
+  (segment (start 193.1 97.8) (end 191.8 97.8) (width 0.5) (layer B.Cu) (net 3))
+  (segment (start 189.8 95.8) (end 189.8 92.35) (width 0.5) (layer B.Cu) (net 3))
+  (segment (start 191.8 97.8) (end 189.8 95.8) (width 0.5) (layer B.Cu) (net 3))
+  (segment (start 187.2 92.3) (end 189.75 92.3) (width 0.5) (layer B.Cu) (net 3))
+  (segment (start 189.75 92.3) (end 189.8 92.35) (width 0.3) (layer B.Cu) (net 3))
   (segment (start 183.642 92.456) (end 183.642 94.158) (width 0.3) (layer F.Cu) (net 3))
   (segment (start 183.642 94.158) (end 181.89 95.91) (width 0.3) (layer F.Cu) (net 3))
@@
   (segment (start 167.64 100.965) (end 168.613 101.938) (width 0.3) (layer F.Cu) (net 3))
   (segment (start 168.613 101.938) (end 169.164 101.938) (width 0.3) (layer F.Cu) (net 3))
-  (segment (start 187.275 92.45) (end 183.648 92.45) (width 0.3) (layer B.Cu) (net 3) (status 10))
+  (segment (start 187.275 92.45) (end 183.648 92.45) (width 0.5) (layer B.Cu) (net 3) (status 10))
   (segment (start 183.648 92.45) (end 183.642 92.456) (width 0.3) (layer B.Cu) (net 3))
   (segment (start 156.64 97.87) (end 156.64 97.89) (width 0.3) (layer F.Cu) (net 3))
@@
   (segment (start 171.28 101.938) (end 171.45 102.108) (width 0.3) (layer F.Cu) (net 3))
   (via (at 171.45 102.108) (size 1.8) (drill 1) (layers F.Cu B.Cu) (net 3))
-  (segment (start 171.45 102.108) (end 181.102 92.456) (width 0.3) (layer B.Cu) (net 3))
-  (segment (start 181.102 92.456) (end 183.642 92.456) (width 0.3) (layer B.Cu) (net 3))
+  (segment (start 171.45 102.108) (end 181.102 92.456) (width 0.5) (layer B.Cu) (net 3))
+  (segment (start 181.102 92.456) (end 183.642 92.456) (width 0.5) (layer B.Cu) (net 3))
   (via (at 183.642 92.456) (size 1.8) (drill 1) (layers F.Cu B.Cu) (net 3))
   (segment (start 180.83 95.91) (end 181.89 95.91) (width 0.3) (layer F.Cu) (net 3))
@@
   (segment (start 164.735 96.565) (end 162.1 99.2) (width 0.3) (layer F.Cu) (net 9))
   (segment (start 162.1 99.2) (end 162.8 99.2) (width 0.25) (layer F.Cu) (net 9) (status 30))
-  (segment (start 193.1 93.3) (end 190.1 93.3) (width 0.3) (layer F.Cu) (net 10))
-  (segment (start 190.1 93.3) (end 189.4 94) (width 0.3) (layer F.Cu) (net 10))
-  (segment (start 182.1 98.515) (end 183.685 98.515) (width 0.3) (layer F.Cu) (net 11))
-  (segment (start 187.2 95) (end 187.2 94) (width 0.3) (layer F.Cu) (net 11))
-  (segment (start 183.685 98.515) (end 187.2 95) (width 0.3) (layer F.Cu) (net 11))
-  (segment (start 178.78 98.515) (end 182.1 98.515) (width 0.3) (layer F.Cu) (net 11))
+  (segment (start 188.5 97.1) (end 189.6 97.1) (width 0.3) (layer F.Cu) (net 10) (status 400000))
+  (segment (start 191.4 95.3) (end 193.1 95.3) (width 0.3) (layer F.Cu) (net 10) (status 800000))
+  (segment (start 189.6 97.1) (end 191.4 95.3) (width 0.3) (layer F.Cu) (net 10))
+  (segment (start 178.78 98.515) (end 182.185 98.515) (width 0.3) (layer F.Cu) (net 11) (status 400000))
+  (segment (start 183.6 97.1) (end 186.3 97.1) (width 0.3) (layer F.Cu) (net 11) (status 800000))
+  (segment (start 182.185 98.515) (end 183.6 97.1) (width 0.3) (layer F.Cu) (net 11))
+  (segment (start 187.4 99.1) (end 187.4 96.1) (width 0.3) (layer F.Cu) (net 12) (status 400000))
+  (segment (start 190.2 93.3) (end 193.1 93.3) (width 0.3) (layer F.Cu) (net 12) (status 800000))
+  (segment (start 187.4 96.1) (end 190.2 93.3) (width 0.3) (layer F.Cu) (net 12))
   (segment (start 187.4 99.1) (end 187.4 99) (width 0.3) (layer F.Cu) (net 12))
-  (segment (start 187.4 99) (end 191.1 95.3) (width 0.3) (layer F.Cu) (net 12))
-  (segment (start 191.1 95.3) (end 193.1 95.3) (width 0.3) (layer F.Cu) (net 12))
   (segment (start 187.4 101.6) (end 187.4 99.1) (width 0.3) (layer F.Cu) (net 12))
   (segment (start 183.7 99.165) (end 185.135 99.165) (width 0.3) (layer F.Cu) (net 13))
